Commit message: top plate pos change

File: scout_description/urdf/decorations.urdf.xacro (robot description, xacro)
@@ -35,6 +35,6 @@
     <xacro:property name="scout_rear_bumper_extend"     value="$(optenv SCOUT_REAR_BUMPER_EXTEND 0)" />
     <xacro:property name="scout_wibotic_bumper_enable"  value="$(optenv SCOUT_WIBOTIC_BUMPER 0)" />
-    <!-- Spawn Husky chassis -->
-    <link name="top_chassis_link">
+    <!-- Spawn chassis: No top chassis in Scout -->
+    <!-- link name="top_chassis_link">
       <visual>
         <origin xyz="0 0 0" rpy="0 0 0" />
@@ -43,11 +43,11 @@
         </geometry>
       </visual>
-    </link>
+    </link -->
     <!-- Attach chassis to the robot -->
-    <joint name="top_chassis_joint" type="fixed">
+    <!-- joint name="top_chassis_joint" type="fixed">
       <parent link="base_link" />
       <child link="top_chassis_link" />
-    </joint>
-    <xacro:if value="$(optenv SCOUT_USER_RAIL_ENABLED true)">
+    </joint -->
+    <xacro:if value="$(optenv SCOUT_USER_RAIL_ENABLED false)">
       <!-- Spawn user rails -->
       <link name="user_rail_link">
@@ -60,5 +60,5 @@
       <!-- Attach user rails to base link -->
       <joint name="user_rail" type="fixed">
-        <origin xyz="0.272 0 0.245" rpy="0 0 0" />
+        <origin xyz="0.24 0 0.12" rpy="0 0 0" />
         <parent link="base_link" />
         <child link="user_rail_link" />
@@ -158,5 +158,5 @@
           <parent link="base_link" />
           <child link="top_plate_link"/>
-          <origin xyz="0.0812 0 0.225" rpy="0 0 0"/>
+          <origin xyz="0 0 0.12" rpy="0 0 0"/>
         </joint>
         <!-- Top plate front link -->
@@ -192,5 +192,5 @@
           <parent link="base_link" />
           <child link="top_plate_link"/>
-          <origin xyz="0.0812 0 0.245" rpy="0 0 0"/>
+          <origin xyz="0 0 0.12" rpy="0 0 0"/>
         </joint>
         <!-- Top plate front link -->

File: scout_description/urdf/scout.urdf.xacro (robot description, xacro)
@@ -22,5 +22,5 @@
     <xacro:arg name="laser_3d_xyz" default="$(optenv SCOUT_LASER_3D_XYZ 0 0 0)" />
     <xacro:arg name="laser_3d_rpy" default="$(optenv SCOUT_LASER_3D_RPY 0 0 0)" />
-    <xacro:arg name="realsense_enabled" default="$(optenv SCOUT_REALSENSE_ENABLED 0)" />
+    <xacro:arg name="realsense_enabled" default="$(optenv SCOUT_REALSENSE_ENABLED 1)" />
     <xacro:arg name="realsense_xyz" default="$(optenv SCOUT_REALSENSE_XYZ 0 0 0)" />
     <xacro:arg name="realsense_rpy" default="$(optenv SCOUT_REALSENSE_RPY 0 0 0)" />
