Commit message: change some husky to scout

File: scout_description/urdf/accessories/hokuyo_ust10.urdf.xacro (robot description, xacro)
@@ -58,5 +58,5 @@
         <geometry>
           <!-- Origin of this mesh is the base of the bracket. -->
-          <mesh filename="package://husky_description/meshes/accessories/hokuyo_ust10.stl" />
+          <mesh filename="package://scout_description/meshes/accessories/hokuyo_ust10.stl" />
         </geometry>
         <material name="dark_grey" />

File: scout_description/urdf/accessories/sensor_arch.urdf.xacro (robot description, xacro)
@@ -8,5 +8,5 @@
              <visual>
                  <geometry>
-                     <mesh filename="package://husky_description/meshes/accessories/${size}_mm_sensor_arch.dae" />
+                     <mesh filename="package://scout_description/meshes/accessories/${size}_mm_sensor_arch.dae" />
                  </geometry>
              </visual>
@@ -14,5 +14,5 @@
                  <origin xyz="0 0 0" rpy="0 0 0"/>
                  <geometry>
-                     <mesh filename="package://husky_description/meshes/accessories/${size}_mm_sensor_arch.dae" />
+                     <mesh filename="package://scout_description/meshes/accessories/${size}_mm_sensor_arch.dae" />
                  </geometry>
              </collision>

File: scout_description/urdf/accessories/sick_lms1xx_mount.urdf.xacro (robot description, xacro)
@@ -33,5 +33,5 @@
         <geometry>
           <!-- Origin of this mesh is the base of the bracket. -->
-          <mesh filename="package://husky_description/meshes/accessories/lms1xx_mount.dae" />
+          <mesh filename="package://scout_description/meshes/accessories/lms1xx_mount.dae" />
         </geometry>
       </visual>

File: scout_description/urdf/wheel.gazebo.xacro (robot description, xacro)
@@ -2,5 +2,5 @@
 <!--
 Software License Agreement (BSD)
-\file      scout_wheel.xacro (adapted from wheel.urdf.xacro in husky_description)
+\file      scout_wheel.xacro (adapted from wheel.urdf.xacro in scout_description)
 \authors   Paul Bovbel <pbovbel@clearpathrobotics.com>
            Ruixiang Du <ruixiang.du@westonrobot.com>

File: scout_description/urdf/wheel.urdf.xacro (robot description, xacro)
@@ -2,5 +2,5 @@
 <!--
 Software License Agreement (BSD)
-\file      scout_wheel.xacro (adapted from wheel.urdf.xacro in husky_description)
+\file      scout_wheel.xacro (adapted from wheel.urdf.xacro in scout_description)
 \authors   Paul Bovbel <pbovbel@clearpathrobotics.com>
            Ruixiang Du <ruixiang.du@westonrobot.com>
