Commit message: remove _g4 postfix

File: scout_description/urdf/accessories/ydlidar.urdf.xacro (robot description, xacro)
@@ -25,5 +25,5 @@
 -->
 <robot xmlns:xacro="http://www.ros.org/wiki/xacro">
-  <xacro:macro name="ydlidar_g4" params="frame:=laser topic:=scan sample_size:=720 update_rate:=50
+  <xacro:macro name="ydlidar" params="frame:=laser topic:=scan sample_size:=720 update_rate:=50
                min_angle:=-2.35619 max_angle:=2.35619 min_range:=0.1 max_range:=30.0 robot_namespace:=/" >
     <link name="${frame}">
@@ -48,5 +48,5 @@
         <geometry>
           <mesh
-            filename="package://scout_description/meshes/accessories/ydlidar_g4.dae" />
+            filename="package://scout_description/meshes/accessories/ydlidar.dae" />
         </geometry>
         <material
@@ -62,5 +62,5 @@
         <geometry>
           <mesh
-            filename="package://scout_description/meshes/accessories/ydlidar_g4.dae" />
+            filename="package://scout_description/meshes/accessories/ydlidar.dae" />
         </geometry>
       </collision>

File: scout_description/urdf/accessories/ydlidar_mount.urdf.xacro (robot description, xacro)
@@ -26,6 +26,6 @@
 -->
 <robot xmlns:xacro="http://ros.org/wiki/xacro">
-  <xacro:include filename="$(find scout_description)/urdf/accessories/ydlidar_g4.urdf.xacro" />
-  <xacro:macro name="ydlidar_g4_mount" params="prefix">
+  <xacro:include filename="$(find scout_description)/urdf/accessories/ydlidar.urdf.xacro" />
+  <xacro:macro name="ydlidar_mount" params="prefix">
     <link name="${prefix}_laser_mount">
       <visual>
@@ -33,5 +33,5 @@
         <geometry>
           <!-- Origin of this mesh is the base of the bracket. -->
-          <mesh filename="package://scout_description/meshes/accessories/ydlidar_g4_mount.dae" />
+          <mesh filename="package://scout_description/meshes/accessories/ydlidar_mount.dae" />
         </geometry>
       </visual>

File: scout_description/urdf/scout.urdf.xacro (robot description, xacro)
@@ -1,7 +1,7 @@
 <?xml version="1.0"?>
 <robot name="scout" xmlns:xacro="http://ros.org/wiki/xacro">
-    <xacro:arg name="laser_enabled" default="$(optenv SCOUT_YDLIDAR_G4_ENABLED 1)" />
-    <xacro:arg name="laser_xyz" default="$(optenv SCOUT_YDLIDAR_G4_XYZ 0.2206 0.0 0.00635)" />
-    <xacro:arg name="laser_rpy" default="$(optenv SCOUT_YDLIDAR_G4_RPY 0.0 0.0 0.0)" />
+    <xacro:arg name="laser_enabled" default="$(optenv SCOUT_YDLIDAR_ENABLED 1)" />
+    <xacro:arg name="laser_xyz" default="$(optenv SCOUT_YDLIDAR_XYZ 0.2206 0.0 0.00635)" />
+    <xacro:arg name="laser_rpy" default="$(optenv SCOUT_YDLIDAR_RPY 0.0 0.0 0.0)" />
     <!--
     <xacro:arg name="laser_enabled" default="$(optenv SCOUT_LMS1XX_ENABLED 0)" />
@@ -44,5 +44,5 @@
     <xacro:include filename="$(find scout_description)/urdf/accessories/intel_realsense.urdf.xacro"/>
     <xacro:include filename="$(find scout_description)/urdf/accessories/sick_lms1xx_mount.urdf.xacro"/>
-    <xacro:include filename="$(find scout_description)/urdf/accessories/ydlidar_g4_mount.urdf.xacro"/>
+    <xacro:include filename="$(find scout_description)/urdf/accessories/ydlidar_mount.urdf.xacro"/>
     <xacro:include filename="$(find scout_description)/urdf/accessories/sensor_arch.urdf.xacro"/>
     <xacro:include filename="$(find scout_description)/urdf/accessories/hokuyo_ust10.urdf.xacro"/>
@@ -164,6 +164,6 @@
         <xacro:sick_lms1xx frame="base_laser" topic="scan" robot_namespace="$(arg robot_namespace)"/>
         -->
-        <xacro:ydlidar_g4_mount prefix="base"/>
-        <xacro:ydlidar_g4 frame="base_laser" topic="scan" robot_namespace="$(arg robot_namespace)"/>
+        <xacro:ydlidar_mount prefix="base"/>
+        <xacro:ydlidar frame="base_laser" topic="scan" robot_namespace="$(arg robot_namespace)"/>
         <joint name="laser_mount_joint" type="fixed">
         <origin xyz="$(arg laser_xyz)" rpy="$(arg laser_rpy)" />
